File: Electronics/HC-OutTemp_revA.sch (EAGLE design)
At the start: 38 parts, among them Q1 16MHz, SW1 SWITCH_SLIDE, U1 ATMEGA328-20P, U2 NRF24L01, U5 BCO35

Commit message: changed: PCB
Parts:
- removed BAT2: 1V5, 1_domaci:BATTERY_1X
- removed C2, C3: 22p, 1_domaci:C-CERAMIC'SMD'
- removed JP1, JP4, JP5, JP6: PINHD-3X1, 1_domaci:PINHD-3X1
- removed Q1: 16MHz, crystal:CRYSTALHC49S
- removed R10, R2, R3, R7: 4K7, 1_domaci:R'2'
- removed R4: 1M, 1_domaci:R'2'
- removed U5: BCO35, 1_domaci:STEP_UP-BCO35
- added U$9: CASE'120X80X40', 1_domaci:CASE'120X80X40'
- added U3: TMP102, 1_domaci:TMP102
- BAT1: value 1V5 -> (none); device 1_domaci:BATTERY_1X -> 1_domaci:BATTERY_1X'DOUBLE'
- LED1: value green -> (none); device 1_domaci:LED'SMD' -> 1_domaci:LED'3MM'
Connections:
- removed net DS18B20_1: JP4.2, R10.P$1, U1.(PCI23/AIN1)PD7
- removed net DS18B20_2: JP1.2, R2.P$1, U1.(PCI0/ICP/CLKO)PB0
- removed net DS18B20_3: JP5.2, R3.P$1, U1.(PCI1/OC1A/OC1S)PB1
- removed net DS18B20_4: JP6.2, R7.P$1, U1.(PCI2/SS/OC1B)PB2
- removed net N$4: C2.P$2, Q1.2, R4.P$2, U1.PB6(XTAL1/TOSC1/PCI6)
- removed net N$8: BAT1.P, BAT2.P, SW1.MIDDLE
- removed net V_BAT: SW1.S, U1.(PCI8/ADC0)PC0, U5.VIN
- new net N$10: U1.(PCI13/ADC5/SCL)PC5, U3.SCL
- new net N$12: U1.(PCI11/ADC3)PC3, U3.ALT
- new net N$9: U1.(PCI12/ADC4/SDA)PC4, U3.SDA
- net +3V3: now also SW1.S, U3.VCC; no longer JP1.1, JP4.1, JP5.1, JP6.1, R10.P$2, R2.P$2, R3.P$2, R7.P$2, U5.VOUT
- net BUT: now also U1.(PCI21/T1/OC0B)PD5; no longer U1.(PCI18/INT0)PD2
- net CE_R: now also U1.(PCI23/AIN1)PD7; no longer U1.(PCI9/ADC1)PC1
- net CS_R: now also U1.(PCI0/ICP/CLKO)PB0; no longer U1.(PCI10/ADC2)PC2
- net GND: now also U3.GND; no longer BAT2.N, C2.P$1, C3.P$1, JP1.3, JP4.3, JP5.3, JP6.3, U5.GND
- net LED: now also U1.(PCI10/ADC2)PC2; no longer U1.(PCI19/INT1/OC2B)PD3
- net N$1: now also BAT1.P, SW1.MIDDLE; no longer C3.P$2, Q1.1, R4.P$1, U1.PB7(XTAL2/TOSC2/PCI7)
Other:
- moved on the sheet: BAT1, BUT1, C5, C6, LED1, R5, R6, R9, SW1, U2

Commit message: changed: MCU package to SMD
Parts:
- added C2: 100n, 1_domaci:C-CERAMIC'SMD'
- U1: value ATMEGA328-20P -> ATMEGA328P-AU; device 1_domaci:ATMEGA328-20P -> 1_domaci:ATMEGA328P-AU
Connections:
- net +3V3: now also C2.P$2
- net BUT: now also U1.(PCI9/ADC1)PC1; no longer U1.(PCI21/T1/OC0B)PD5
- net CE_R: now also U1.(PCI2/SS/OC1B)PB2; no longer U1.(PCI23/AIN1)PD7
- net CS_R: now also U1.(PCI1/OC1A/OC1S)PB1; no longer U1.(PCI0/ICP/CLKO)PB0
- net GND: now also C2.P$1, U1.(PCI0/ICP/CLKO)PB0, U1.ADC6

Commit message: modified: PCB
Parts:
- added R2: 0R, 1_domaci:R'2'
- BAT1: value (none) -> 2xAA
- R9: value 1K -> ?K
Connections:
- new net N$8: JP3.2, R2.P$2
- net RX: now also R2.P$1; no longer JP3.2
Other:
- moved on the sheet: BAT1, BUT1, C1, C2, C4, C5, C6, JP2, JP3, LED1, R1, R5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

Commit message: modified: PCB
Parts:
- R9: value ?K -> 4k7
Changed lines of the file:
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@@
 <part name="U$7" library="1_domaci" deviceset="HOLE" device=""/>
 <part name="U$8" library="1_domaci" deviceset="HOLE" device=""/>
-<part name="R9" library="1_domaci" deviceset="R" device="'2'" value="?K"/>
+<part name="R9" library="1_domaci" deviceset="R" device="'2'" value="4k7"/>
 <part name="GND13" library="supply1" deviceset="GND" device=""/>
 <part name="GND15" library="supply1" deviceset="GND" device=""/>
